File: main_pcb/kicad_docs/bit_crusher_pedal.kicad_pcb (KiCad board)
At the start: 2 copper layers, 81.3 x 61 mm, 70 parts, among them J1 audio_input, J2 audio_output, J3 SWD_header, J4 9v_DC_in, J5 extern_resolution_CV, J6 extern_sample_rate_CV, J7 to_LED, U1 MCP6002-xP, U2 MCP6002-xP, U3 STM32F334K6Tx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

Commit message: add compander
Parts:
- added C27: 220nF, Capacitor_SMD:C_0805_2012Metric_Pad1.15x1.40mm_HandSolder, B.Cu at (135.5, 74.9)
- added C28: 220pF, Capacitor_SMD:C_0805_2012Metric_Pad1.15x1.40mm_HandSolder, B.Cu at (135.4, 87.6)
- added C29: 10uF, Capacitor_SMD:C_0805_2012Metric_Pad1.15x1.40mm_HandSolder, B.Cu at (135.5, 90.2)
- added C30: 220nF, Capacitor_SMD:C_0805_2012Metric_Pad1.15x1.40mm_HandSolder, B.Cu at (152.7, 85.1)
- added C31: 220pF, Capacitor_SMD:C_0805_2012Metric_Pad1.15x1.40mm_HandSolder, B.Cu at (152.7, 92.7)
- added C32: 220nF, Capacitor_SMD:C_0805_2012Metric_Pad1.15x1.40mm_HandSolder, B.Cu at (152.7, 74.9)
- added C33: 10uF, Capacitor_SMD:C_0805_2012Metric_Pad1.15x1.40mm_HandSolder, B.Cu at (152.7, 80.0)
- added C34: 2.2uF, Capacitor_SMD:C_0805_2012Metric_Pad1.15x1.40mm_HandSolder, B.Cu at (152.7, 90.2)
- added C35: 10uF, Capacitor_SMD:C_0805_2012Metric_Pad1.15x1.40mm_HandSolder, B.Cu at (140.1, 72.4)
- added C36: 100nF, Capacitor_SMD:C_0805_2012Metric_Pad1.15x1.40mm_HandSolder, B.Cu at (140.1, 74.9)
- added C37: 10nF, Capacitor_SMD:C_0805_2012Metric_Pad1.15x1.40mm_HandSolder, B.Cu at (142.5, 98.3)
- added Q1: MMBF5457, Package_TO_SOT_SMD:SOT-23_Handsoldering, B.Cu at (147.8, 98.3)
- added R24: opt, Resistor_SMD:R_0805_2012Metric_Pad1.15x1.40mm_HandSolder, B.Cu at (135.4, 82.5)
- added R25: 560, Resistor_SMD:R_0805_2012Metric_Pad1.15x1.40mm_HandSolder, B.Cu at (135.4, 85.1)
- added R26: 1M, Resistor_SMD:R_0805_2012Metric_Pad1.15x1.40mm_HandSolder, B.Cu at (135.5, 92.7)
- added R27: 22k, Resistor_SMD:R_0805_2012Metric_Pad1.15x1.40mm_HandSolder, B.Cu at (152.7, 82.5)
- added R28: 2M2, Resistor_SMD:R_0805_2012Metric_Pad1.15x1.40mm_HandSolder, B.Cu at (152.7, 72.4)
- added R29: 22k, Resistor_SMD:R_0805_2012Metric_Pad1.15x1.40mm_HandSolder, B.Cu at (152.7, 87.6)
- added R30: 10k, Resistor_SMD:R_0805_2012Metric_Pad1.15x1.40mm_HandSolder, B.Cu at (152.7, 77.5)
- added R31: 2M2, Resistor_SMD:R_0805_2012Metric_Pad1.15x1.40mm_HandSolder, B.Cu at (142.5, 101.3)
- added R32: 2M2, Resistor_SMD:R_0805_2012Metric_Pad1.15x1.40mm_HandSolder, B.Cu at (147.3, 94.7)
- added R33: 2M2, Resistor_SMD:R_0805_2012Metric_Pad1.15x1.40mm_HandSolder, B.Cu at (149.1, 101.3)
- added R34: 10k, Resistor_SMD:R_0805_2012Metric_Pad1.15x1.40mm_HandSolder, B.Cu at (152.4, 100.3)
- added RV4: 100k, Potentiometer_THT:Potentiometer_Bourns_3296W_Vertical, B.Cu at (88.9, 76.2)
- added RV5: 100k, Potentiometer_THT:Potentiometer_Bourns_3296W_Vertical, B.Cu at (88.9, 86.4)
- added U5: NE570, Package_SO:SOIC-16W_7.5x10.3mm_P1.27mm, B.Cu at (144.0, 83.2)
- C4: value 220nF -> 47nF; footprint Capacitor_THT:C_Rect_L7.0mm_W3.5mm_P5.00mm -> Capacitor_SMD:C_0805_2012Metric_Pad1.15x1.40mm_HandSolder
- C8: value 10uF -> 470nF; footprint Capacitor_THT:CP_Radial_D6.3mm_P2.50mm -> Capacitor_SMD:C_0805_2012Metric_Pad1.15x1.40mm_HandSolder
- R11: value 560 -> 10k
- R12: value 1M -> 2M2
- R15, R19: value selec -> 10k
- R16, R20: value 120k -> 100k
- R17, R18, R21, R22: value 82k -> 68k
- R5: value 1M -> 22k
- R6: value 390k -> 100k
- moved J1 36.8 mm to (142.9, 109.2), turned to 270 degrees
- moved J2 31.0 mm to (134.6, 109.2), turned to 270 degrees
- moved R23 24.5 mm to (118.4, 104.4)
- moved C4 24.4 mm to (118.1, 77.0), turned to 270 degrees
- moved R12 21.5 mm to (135.5, 72.4), turned to 0 degrees
- moved J7 20.3 mm to (121.9, 109.2)
- moved R11 14.6 mm to (135.4, 77.5)
- moved R13 13.3 mm to (115.4, 98.8)
- moved R14 13.3 mm to (121.2, 98.8)
- moved C22 13.3 mm to (118.4, 98.8)
- moved R5 13.0 mm to (141.2, 66.0)
- moved C23 10.7 mm to (115.6, 77.0)
- moved C25 10.7 mm to (115.6, 89.7)
- moved C26 10.7 mm to (104.1, 89.7)
- moved R10 10.7 mm to (123.2, 89.7)
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Connections:
- C4 pad 2: /audio_input/dry_audio_input -> /variable_gain_amp/audio_in
- C6 pad 1: Net-(C6-Pad1) -> /expander/expander_in
- C8 pad 2: /audio_output/buffered_wet_audio -> /expander/expander_in
- J1 pad 1: /audio_input/dry_audio_input -> /compressor/compressor_in
- J2 pad 1: /audio_output/buffered_wet_audio -> /expander/expander_out
- R11 pad 1: Net-(C8-Pad1) -> Net-(R11-Pad1)
- R11 pad 2: Net-(C6-Pad1) -> Net-(C8-Pad1)
- R12 pad 1: GND -> +9V
- R12 pad 2: /audio_output/buffered_wet_audio -> Net-(C27-Pad2)
- R15 pad 1: +9V -> Net-(R15-Pad1)
- R19 pad 1: +9V -> Net-(R19-Pad1)
- R5 pad 1: GND -> Net-(R5-Pad1)
- R5 pad 2: /audio_input/dry_audio_input -> Net-(R5-Pad2)
- R6 pad 1: Net-(R6-Pad1) -> Net-(R5-Pad2)
- RV1 pad : (no net) -> GND
- RV1 pad 1: Net-(R6-Pad1) -> Net-(R5-Pad1)
- RV2 pad : (no net) -> GND
- RV3 pad : (no net) -> GND
- U1 pad 2: Net-(R6-Pad1) -> Net-(R5-Pad2)
- U1 pad 6: Net-(C6-Pad1) -> /expander/expander_in
- U1 pad 7: Net-(C6-Pad1) -> /expander/expander_in
Routing:
- net +9V: track 57.4 -> 130.1 mm, vias 3 -> 2
- net /variable_gain_amp/audio_in: track 0.00 -> 65.7 mm, vias 0 -> 2
- net +3V3: track 193.9 -> 153.8 mm, vias 12 -> 8
- net Net-(R5-Pad2): track 0.00 -> 34.2 mm, vias 0 -> 2
- net Net-(R6-Pad1): track 27.6 -> 0.00 mm, vias 2 -> 0
- net Net-(C6-Pad1): track 24.6 -> 0.00 mm
- net /expander/expander_in: track 0.00 -> 24.2 mm, vias 0 -> 4
- net Net-(C30-Pad2): track 0.00 -> 23.3 mm, vias 0 -> 2
- net /expander/expander_out: track 0.00 -> 22.2 mm, vias 0 -> 1
- net Net-(C34-Pad1): track 0.00 -> 20.7 mm
- net Net-(R3-Pad2): track 63.4 -> 80.6 mm
- net GND: track 28.4 -> 12.3 mm, vias 58 -> 74
- net Net-(C23-Pad1): track 50.0 -> 38.2 mm, vias 1 -> 0
- net /compressor/compressor_in: track 0.00 -> 11.5 mm
- net Net-(C4-Pad1): track 14.0 -> 2.55 mm
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Other:
- board text added: "bit CV trim"
- board text added: "github.com/JordanAceto/bit_crusher_pedal rev 1 2020-08-17"
- board text added: "rate CV trim"
- board text removed: "Bit crusher rev 0 2020-07-27"
