File: main_pcb/kicad_docs/bit_crusher_pedal.sch (KiCad schematic (older format))
At the start: 4 parts, among them J1 audio_input, J2 audio_output

Commit message: add compander
Connections:
- net audio_input/dry_audio_input renamed compressor/compressor_in
- net audio_output/buffered_wet_audio renamed expander/expander_out
Other:
- moved on the sheet: H1, H2, J1, J2
Changed lines of the file:
@@
 $Descr A4 11693 8268
 encoding utf-8
-Sheet 1 6
+Sheet 1 8
 Title "Bit Crusher Pedal"
-Date "2020-07-27"
-Rev "0"
+Date "2020-08-16"
+Rev "1"
 Comp ""
 Comment1 "creativecommons.org/licenses/by/4.0/"
@@
 $EndDescr
 $Sheet
-S 5000 1500 1500 1500
+S 5000 2050 1500 1500
 U 5F120841
 F0 "microcontroller" 50
 F1 "microcontroller.sch" 50
-F2 "DAC_out" O R 6500 1650 50
-F3 "resolution_CV_in" I L 5000 2700 50
-F4 "sample_rate_CV_in" I L 5000 2850 50
-F5 "ADC_in" I L 5000 1650 50
-$EndSheet
-$Sheet
-S 2500 1500 1500 1500
-U 5F122414
-F0 "audio_input" 50
-F1 "audio_input.sch" 50
-F2 "buffered_dry_audio" O R 4000 1650 50
-F3 "dry_audio_input" I L 2500 1650 50
-$EndSheet
-$Sheet
-S 7500 1500 1500 1500
-U 5F122464
-F0 "audio_output" 50
-F1 "audio_output.sch" 50
-F2 "wet_from_DAC" I L 7500 1650 50
-F3 "buffered_wet_audio" O R 9000 1650 50
-$EndSheet
-$Sheet
-S 7500 3500 1500 1500
+F2 "DAC_out" O R 6500 2550 50
+F3 "resolution_CV_in" I L 5000 3250 50
+F4 "sample_rate_CV_in" I L 5000 3400 50
+F5 "ADC_in" I L 5000 2200 50
+$EndSheet
+$Sheet
+S 7000 4050 1500 1500
 U 5F1224B4
 F0 "power_supply" 50
 F1 "power_supply.sch" 50
 $EndSheet
-$Sheet
-S 5000 3500 1500 1500
+$Comp
+L Connector_Generic:Conn_01x02 J1
+U 1 1 5F242118
+P 1050 2200
+F 0 "J1" H 968 2417 50  0000 C CNN
+F 1 "audio_input" H 968 2326 50  0000 C CNN
+F 2 "Connector_PinHeader_2.54mm:PinHeader_1x02_P2.54mm_Vertical" H 1050 2200 50  0001 C CNN
+F 3 "~" H 1050 2200 50  0001 C CNN
+	1    1050 2200
+	-1   0    0    -1
+$EndComp
+$Comp
+L power:GND #PWR0101
+U 1 1 5F2427AB
+P 1350 2400
+F 0 "#PWR0101" H 1350 2150 50  0001 C CNN
+F 1 "GND" H 1355 2227 50  0000 C CNN
+F 2 "" H 1350 2400 50  0001 C CNN
+F 3 "" H 1350 2400 50  0001 C CNN
+	1    1350 2400
+	1    0    0    -1
+$EndComp
+Wire Wire Line
+	1350 2400 1350 2300
+Wire Wire Line
+	1350 2300 1250 2300
+Wire Wire Line
+	10150 2450 10150 2350
+Wire Wire Line
+	5000 4200 4900 4200
+Wire Wire Line
+	4900 4200 4900 3250
+Wire Wire Line
+	4900 3250 5000 3250
+Wire Wire Line
+	5000 3400 4800 3400
+Wire Wire Line
+	4800 3400 4800 4350
+Wire Wire Line
+	4800 4350 5000 4350
+$Comp
+L Mechanical:MountingHole_Pad H2
+U 1 1 5F20120B
+P 6000 7300
+F 0 "H2" H 6100 7349 50  0000 L CNN
+F 1 "MountingHole_Pad" H 6100 7258 50  0000 L CNN
+F 2 "MountingHole:MountingHole_3.2mm_M3_Pad_Via" H 6000 7300 50  0001 C CNN
+F 3 "~" H 6000 7300 50  0001 C CNN
+	1    6000 7300
+	1    0    0    -1
+$EndComp
+$Comp
+L power:GND #PWR02
+U 1 1 5F201718
+P 6000 7400
+F 0 "#PWR02" H 6000 7150 50  0001 C CNN
+F 1 "GND" H 6005 7227 50  0000 C CNN
+F 2 "" H 6000 7400 50  0001 C CNN
+F 3 "" H 6000 7400 50  0001 C CNN
+	1    6000 7400
+	1    0    0    -1
+$EndComp
+$Comp
+L Mechanical:MountingHole_Pad H1
+U 1 1 5F201A9A
+P 6000 6800
+F 0 "H1" H 6100 6849 50  0000 L CNN
+F 1 "MountingHole_Pad" H 6100 6758 50  0000 L CNN
+F 2 "MountingHole:MountingHole_3.2mm_M3_Pad_Via" H 6000 6800 50  0001 C CNN
+F 3 "~" H 6000 6800 50  0001 C CNN
+	1    6000 6800
+	1    0    0    -1
+$EndComp
+$Comp
+L power:GND #PWR01
+U 1 1 5F201AA0
+P 6000 6900
+F 0 "#PWR01" H 6000 6650 50  0001 C CNN
+F 1 "GND" H 6005 6727 50  0000 C CNN
+F 2 "" H 6000 6900 50  0001 C CNN
+F 3 "" H 6000 6900 50  0001 C CNN
+	1    6000 6900
+	1    0    0    -1
+$EndComp
+$Sheet
+S 8500 2050 1000 1050
+U 5F3D7D32
+F0 "expander" 50
+F1 "expander.sch" 50
+F2 "expander_in" I L 8500 2250 50
+F3 "expander_out" O R 9500 2600 50
+$EndSheet
+Wire Wire Line
+	10150 2350 10250 2350
+$Comp
+L power:GND #PWR0102
+U 1 1 5F243C9B
+P 10150 2450
+F 0 "#PWR0102" H 10150 2200 50  0001 C CNN
+F 1 "GND" H 10155 2277 50  0000 C CNN
+F 2 "" H 10150 2450 50  0001 C CNN
+F 3 "" H 10150 2450 50  0001 C CNN
+	1    10150 2450
+	-1   0    0    -1
+$EndComp
+$Comp
+L Connector_Generic:Conn_01x02 J2
+U 1 1 5F243C95
+P 10450 2250
+F 0 "J2" H 10400 2500 50  0000 L CNN
+F 1 "audio_output" H 10200 2400 50  0000 L CNN
+F 2 "Connector_PinHeader_2.54mm:PinHeader_1x02_P2.54mm_Vertical" H 10450 2250 50  0001 C CNN
+F 3 "~" H 10450 2250 50  0001 C CNN
+	1    10450 2250
+	1    0    0    -1
+$EndComp
+$Sheet
+S 7000 2050 1000 1000
+U 5F122464
+F0 "low_pass_filter" 50
+F1 "low_pass_filter.sch" 50
+F2 "wet_from_DAC" I L 7000 2200 50
+F3 "low_passed_wet_signal" O R 8000 2550 50
+$EndSheet
+Wire Wire Line
+	1250 2200 2000 2200
+$Sheet
+S 3500 2050 1000 1000
+U 5F122414
+F0 "variable_gain_amp" 50
+F1 "variable_gain_amp.sch" 50
+F2 "audio_in" I L 3500 2200 50
+F3 "scaled_audio_out" O R 4500 2550 50
+$EndSheet
+$Sheet
+S 2000 2000 1000 1050
+U 5F3D7CC8
+F0 "compressor" 50
+F1 "compressor.sch" 50
+F2 "compressor_out" O R 3000 2550 50
+F3 "compressor_in" I L 2000 2200 50
+$EndSheet
+Wire Wire Line
+	3000 2550 3250 2550
+Wire Wire Line
+	3250 2550 3250 2200
+Wire Wire Line
+	3250 2200 3500 2200
+Wire Wire Line
+	4500 2550 4750 2550
+Wire Wire Line
+	4750 2550 4750 2200
+Wire Wire Line
+	4750 2200 5000 2200
+Wire Wire Line
+	6500 2550 6750 2550
+Wire Wire Line
+	6750 2550 6750 2200
+Wire Wire Line
+	6750 2200 7000 2200
+Wire Wire Line
+	8000 2550 8250 2550
+Wire Wire Line
+	8250 2550 8250 2250
+Wire Wire Line
+	8250 2250 8500 2250
+$Sheet
+S 5000 4050 1500 1500
 U 5F1223E3
 F0 "control_voltage_generator" 50
 F1 "control_voltage_generator.sch" 50
-F2 "resolution_CV_out" O L 5000 3650 50
-F3 "sample_rate_CV_out" O L 5000 3800 50
-$EndSheet
-$Comp
-L Connector_Generic:Conn_01x02 J1
-U 1 1 5F242118
-P 1500 1650
-F 0 "J1" H 1418 1867 50  0000 C CNN
-F 1 "audio_input" H 1418 1776 50  0000 C CNN
-F 2 "Connector_PinHeader_2.54mm:PinHeader_1x02_P2.54mm_Vertical" H 1500 1650 50  0001 C CNN
-F 3 "~" H 1500 1650 50  0001 C CNN
-	1    1500 1650
-	-1   0    0    -1
-$EndComp
-$Comp
-L power:GND #PWR0101
-U 1 1 5F2427AB
-P 1800 1850
-F 0 "#PWR0101" H 1800 1600 50  0001 C CNN
-F 1 "GND" H 1805 1677 50  0000 C CNN
-F 2 "" H 1800 1850 50  0001 C CNN
-F 3 "" H 1800 1850 50  0001 C CNN
-	1    1800 1850
-	1    0    0    -1
-$EndComp
-Wire Wire Line
-	1800 1850 1800 1750
-Wire Wire Line
-	1800 1750 1700 1750
-Wire Wire Line
-	1700 1650 2500 1650
-$Comp
-L Connector_Generic:Conn_01x02 J2
-U 1 1 5F243C95
-P 10000 1650
-F 0 "J2" H 9950 1900 50  0000 L CNN
-F 1 "audio_output" H 9750 1800 50  0000 L CNN
-F 2 "Connector_PinHeader_2.54mm:PinHeader_1x02_P2.54mm_Vertical" H 10000 1650 50  0001 C CNN
-F 3 "~" H 10000 1650 50  0001 C CNN
-	1    10000 1650
-	1    0    0    -1
-$EndComp
-$Comp
-L power:GND #PWR0102
-U 1 1 5F243C9B
-P 9700 1850
-F 0 "#PWR0102" H 9700 1600 50  0001 C CNN
-F 1 "GND" H 9705 1677 50  0000 C CNN
-F 2 "" H 9700 1850 50  0001 C CNN
-F 3 "" H 9700 1850 50  0001 C CNN
-	1    9700 1850
-	-1   0    0    -1
-$EndComp
-Wire Wire Line
-	9700 1850 9700 1750
-Wire Wire Line
-	9700 1750 9800 1750
-Wire Wire Line
-	9800 1650 9000 1650
-Wire Wire Line
-	4000 1650 5000 1650
-Wire Wire Line
-	6500 1650 7500 1650
-Wire Wire Line
-	5000 3650 4900 3650
-Wire Wire Line
-	4900 3650 4900 2700
-Wire Wire Line
-	4900 2700 5000 2700
-Wire Wire Line
-	5000 2850 4800 2850
-Wire Wire Line
-	4800 2850 4800 3800
-Wire Wire Line
-	4800 3800 5000 3800
-$Comp
-L Mechanical:MountingHole_Pad H2
-U 1 1 5F20120B
-P 10000 5550
-F 0 "H2" H 10100 5599 50  0000 L CNN
-F 1 "MountingHole_Pad" H 10100 5508 50  0000 L CNN
-F 2 "MountingHole:MountingHole_3.2mm_M3_Pad_Via" H 10000 5550 50  0001 C CNN
-F 3 "~" H 10000 5550 50  0001 C CNN
-	1    10000 5550
-	1    0    0    -1
-$EndComp
-$Comp
-L power:GND #PWR02
-U 1 1 5F201718
-P 10000 5650
-F 0 "#PWR02" H 10000 5400 50  0001 C CNN
-F 1 "GND" H 10005 5477 50  0000 C CNN
-F 2 "" H 10000 5650 50  0001 C CNN
-F 3 "" H 10000 5650 50  0001 C CNN
-	1    10000 5650
-	1    0    0    -1
-$EndComp
-$Comp
-L Mechanical:MountingHole_Pad H1
-U 1 1 5F201A9A
-P 10000 5050
-F 0 "H1" H 10100 5099 50  0000 L CNN
-F 1 "MountingHole_Pad" H 10100 5008 50  0000 L CNN
-F 2 "MountingHole:MountingHole_3.2mm_M3_Pad_Via" H 10000 5050 50  0001 C CNN
-F 3 "~" H 10000 5050 50  0001 C CNN
-	1    10000 5050
-	1    0    0    -1
-$EndComp
-$Comp
-L power:GND #PWR01
-U 1 1 5F201AA0
-P 10000 5150
-F 0 "#PWR01" H 10000 4900 50  0001 C CNN
-F 1 "GND" H 10005 4977 50  0000 C CNN
-F 2 "" H 10000 5150 50  0001 C CNN
-F 3 "" H 10000 5150 50  0001 C CNN
-	1    10000 5150
-	1    0    0    -1
-$EndComp
+F2 "resolution_CV_out" O L 5000 4200 50
+F3 "sample_rate_CV_out" O L 5000 4350 50
+$EndSheet
+Wire Wire Line
+	9500 2600 9750 2600
+Wire Wire Line
+	9750 2600 9750 2250
+Wire Wire Line
+	9750 2250 10250 2250
 $EndSCHEMATC
