File: main_pcb/kicad_docs/power_supply.sch (KiCad schematic (older format))
At the start: 22 parts, among them J4 9v_DC_in, J7 to_LED, U1 MCP6002-xP, U2 MCP6002-xP, U4 AMS1117-3.3

Commit message: add compander
Parts:
- added C35: 10uF, Capacitor_SMD:C_0805_2012Metric_Pad1.15x1.40mm_HandSolder, symbol Device:C
- added C36: 100nF, Capacitor_SMD:C_0805_2012Metric_Pad1.15x1.40mm_HandSolder, symbol Device:C
- added U5: NE570, Package_SO:SOIC-16W_7.5x10.3mm_P1.27mm, symbol compander_parts:NE570
Connections:
- net +9V: now also C35.1, C36.1, U5.13 (Vcc)
- net GND: now also C35.2, C36.2, U5.4 (gnd)
Other:
- note added: "NE570 decoupling"
- note added: "NE570 power"
- moved on the sheet: C10, C11, C12, C13, C14, C15, C16, C17, C18, C19, C20, C21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
