File: main_pcb/kicad_docs/variable_gain_amp.sch (KiCad schematic (older format))
At the start: 8 parts, among them U1 MCP6002-xP

Commit message: add compander
Parts:
- C4: value 220nF -> 47nF; footprint Capacitor_THT:C_Rect_L7.0mm_W3.5mm_P5.00mm -> Capacitor_SMD:C_0805_2012Metric_Pad1.15x1.40mm_HandSolder
- R5: value 1M -> 22k
- R6: value 390k -> 100k
Connections:
- net GND: no longer R5.1
- net at R6.1, U1.2 (-): now also R5.2; no longer RV1.1
- net buffered_dry_audio renamed scaled_audio_out
- net dry_audio_input renamed audio_in
- net audio_in: no longer R5.2
- new net: R5.1, RV1.1
Other:
- note removed: "Variable gain input amplifier"
- moved on the sheet: RV1
Changed lines of the file:
@@
 $Descr A4 11693 8268
 encoding utf-8
-Sheet 3 7
+Sheet 6 8
 Title "Bit Crusher Pedal"
-Date "2020-07-27"
-Rev "0"
+Date "2020-08-16"
+Rev "1"
 Comp ""
 Comment1 "creativecommons.org/licenses/by/4.0/"
@@
 AR Path="/5F122414/5F1F7EDD" Ref="R6"  Part="1"
 F 0 "R6" V 5150 3500 50  0000 L CNN
-F 1 "390k" V 5250 3450 50  0000 L CNN
+F 1 "100k" V 5250 3450 50  0000 L CNN
 F 2 "Resistor_SMD:R_0805_2012Metric_Pad1.15x1.40mm_HandSolder" V 5180 3550 50  0001 C CNN
 F 3 "~" H 5250 3550 50  0001 C CNN
@@
 $EndComp
 Wire Wire Line
-	5700 3300 5500 3300
-Wire Wire Line
 	5500 3300 5500 3550
 Wire Wire Line
 	5500 3550 5600 3550
 Wire Wire Line
-	6200 3650 6250 3650
+	6200 3650 6550 3650
 Wire Wire Line
-	6250 3650 6250 3300
+	6550 3650 6550 3300
 Wire Wire Line
-	6250 3300 6100 3300
+	6550 3300 6400 3300
 Connection ~ 5500 3550
 $Comp
@@
 	5000 4100 5000 4200
 Text HLabel 4500 3550 0    50   Input ~ 0
-dry_audio_input
-Wire Wire Line
-	4700 3550 4600 3550
+audio_in
 Wire Wire Line
 	5000 3550 5100 3550
-Text HLabel 6250 3550 2    50   Output ~ 0
-buffered_dry_audio
+Text HLabel 6550 3550 2    50   Output ~ 0
+scaled_audio_out
 $Comp
 L Device:C C4
@@
 P 4850 3550
 F 0 "C4" V 4598 3550 50  0000 C CNN
-F 1 "220nF" V 4689 3550 50  0000 C CNN
-F 2 "Capacitor_THT:C_Rect_L7.0mm_W3.5mm_P5.00mm" H 4888 3400 50  0001 C CNN
+F 1 "47nF" V 4689 3550 50  0000 C CNN
+F 2 "Capacitor_SMD:C_0805_2012Metric_Pad1.15x1.40mm_HandSolder" H 4888 3400 50  0001 C CNN
 F 3 "~" H 4850 3550 50  0001 C CNN
 	1    4850 3550
@@
 L Device:R_POT RV1
 U 1 1 5F20CAF4
-P 5850 3300
-F 0 "RV1" V 6050 3550 50  0000 C CNN
-F 1 "1M" V 5850 3300 50  0000 C CNN
-F 2 "Potentiometer_THT:Potentiometer_Alpha_RD901F-40-00D_Single_Vertical" H 5850 3300 50  0001 C CNN
-F 3 "~" H 5850 3300 50  0001 C CNN
-	1    5850 3300
+P 6150 3300
+F 0 "RV1" V 6350 3450 50  0000 C CNN
+F 1 "1M" V 6150 3300 50  0000 C CNN
+F 2 "Potentiometer_THT:Potentiometer_Alpha_RD901F-40-00D_Single_Vertical" H 6150 3300 50  0001 C CNN
+F 3 "~" H 6150 3300 50  0001 C CNN
+	1    6150 3300
 	0    -1   -1   0
 $EndComp
 Wire Wire Line
-	5850 3150 5850 3050
+	6150 3150 6150 3050
 Wire Wire Line
-	5850 3050 6100 3050
+	6150 3050 6400 3050
 Wire Wire Line
-	6100 3050 6100 3300
-Connection ~ 6100 3300
+	6400 3050 6400 3300
+Connection ~ 6400 3300
 Wire Wire Line
-	6100 3300 6000 3300
-Text Notes 5500 3250 0    50   ~ 0
+	6400 3300 6300 3300
+Text Notes 6250 3000 0    50   ~ 0
 gain
-Text Notes 3750 2650 0    157  ~ 0
-Variable gain input amplifier
 $Comp
 L Device:R R?
-U 1 1 5F2AE6A2
-P 4600 3800
-AR Path="/5F1223E3/5F2AE6A2" Ref="R?"  Part="1"
-AR Path="/5F122414/5F2AE6A2" Ref="R5"  Part="1"
-F 0 "R5" H 4450 3800 50  0000 L CNN
-F 1 "1M" V 4600 3750 50  0000 L CNN
-F 2 "Resistor_SMD:R_0805_2012Metric_Pad1.15x1.40mm_HandSolder" V 4530 3800 50  0001 C CNN
-F 3 "~" H 4600 3800 50  0001 C CNN
-	1    4600 3800
-	-1   0    0    1
+U 1 1 5F3ABCDA
+P 5750 3300
+AR Path="/5F1223E3/5F3ABCDA" Ref="R?"  Part="1"
+AR Path="/5F122414/5F3ABCDA" Ref="R5"  Part="1"
+F 0 "R5" V 5650 3250 50  0000 L CNN
+F 1 "22k" V 5750 3200 50  0000 L CNN
+F 2 "Resistor_SMD:R_0805_2012Metric_Pad1.15x1.40mm_HandSolder" V 5680 3300 50  0001 C CNN
+F 3 "~" H 5750 3300 50  0001 C CNN
+	1    5750 3300
+	0    1    1    0
 $EndComp
 Wire Wire Line
-	4600 3650 4600 3550
+	5900 3300 6000 3300
 Wire Wire Line
-	4600 3550 4500 3550
-Connection ~ 4600 3550
-$Comp
-L power:GND #PWR0115
-U 1 1 5F2B11E6
-P 4600 3950
-F 0 "#PWR0115" H 4600 3700 50  0001 C CNN
-F 1 "GND" H 4605 3777 50  0000 C CNN
-F 2 "" H 4600 3950 50  0001 C CNN
-F 3 "" H 4600 3950 50  0001 C CNN
-	1    4600 3950
-	1    0    0    -1
-$EndComp
+	5600 3300 5500 3300
+Wire Wire Line
+	4500 3550 4700 3550
 $EndSCHEMATC
