File: hardware/main_pcb/kicad_docs/bit_crusher_pedal.kicad_pcb (KiCad board)
At the start: 2 copper layers, 81.3 x 61 mm, 96 parts, among them J1 audio_input, J2 audio_output, J3 SWD_header, J4 9v_DC_in, J5 extern_resolution_CV, J6 extern_sample_rate_CV, J7 to_LED, Q1 MMBF5457, U1 MCP6002-xP, U2 MCP6002-xP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

Commit message: add rev 1 main pcb docs
Other:
- board text added: "bit-CV in"
- board text added: "bit-CV trim"
- board text added: "rate-CV in"
- board text added: "rate-CV trim"
- board text removed: "bit CV trim"
- board text removed: "bit depth CV in"
- board text removed: "rate CV trim"
- board text removed: "sample-rate CV in"
